File: Batterycharger005.brd (EAGLE design)
At the start: 106 parts

Commit message: Add files via upload
Parts:
- moved E$4 0.79 mm to (-15.9, -33.2), turned to 90 degrees
- moved E$5 0.16 mm to (-15.9, -48.7), turned to 90 degrees
Connections:
- net S$126 renamed S$96
- net S$80 renamed S$60
- net S$100: now also E$5.16; no longer E$5.7
- net S$11: now also E$4.6; no longer E$4.15
- net S$2: now also E$4.10; no longer E$4.1
- net S$3: now also E$4.11; no longer E$4.2
- net S$32: now also E$4.5; no longer E$4.14
- net S$37: now also E$4.4; no longer E$4.13
- net S$38: now also E$4.3; no longer E$4.12
- net S$39: now also E$4.2; no longer E$4.11
- net S$4: now also E$4.12; no longer E$4.3
- net S$40: now also E$4.16; no longer E$4.7
- net S$41: now also E$5.10; no longer E$5.1
- net S$42: now also E$5.11; no longer E$5.2
- net S$43: now also E$5.12; no longer E$5.3
- net S$44: now also E$5.13; no longer E$5.4
- net S$5: now also E$4.13; no longer E$4.4
- net S$61: now also E$5.14; no longer E$5.5
- net S$62: now also E$4.1; no longer E$4.10
- net S$65: now also E$5.7; no longer E$5.16
- net S$66: now also E$5.6; no longer E$5.15
- net S$67: now also E$5.5; no longer E$5.14
- net S$68: now also E$5.4; no longer E$5.13
- net S$69: now also E$5.3; no longer E$5.12
- net S$7: now also E$4.14; no longer E$4.5
- net S$70: now also E$5.2; no longer E$5.11
- net S$71: now also E$5.1; no longer E$5.10
- net S$8: now also E$4.15; no longer E$4.6
- net S$9: now also E$4.7; no longer E$4.16
- net S$99: now also E$5.15; no longer E$5.6
Routing:
- net S$60: track 764.2 -> 727.3 mm, vias 8 -> 6
- net S$96: track 679.9 -> 646.9 mm
- net S$71: track 79.0 -> 59.4 mm
- net S$70: track 82.0 -> 63.4 mm
- net S$69: track 79.0 -> 61.6 mm
- net S$68: track 82.0 -> 66.3 mm
- net S$41: track 172.8 -> 157.8 mm
- net S$67: track 79.0 -> 64.5 mm
- net S$42: track 176.4 -> 163.1 mm
- net S$66: track 82.0 -> 68.8 mm
- net S$65: track 79.0 -> 67.3 mm
- net S$43: track 182.4 -> 171.0 mm
- net S$4: track 143.7 -> 132.6 mm
- net S$5: track 147.3 -> 137.1 mm
- net S$44: track 189.0 -> 179.4 mm
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